File: board/maclight-v2.sch (EAGLE design)
At the start: 28 parts, among them IC1 AT90S2313S, U2 STP16CP05SO-24, Y1 FA-128

Commit message: Trying out attiny85 version
Parts:
- removed C3: 0.1uF, SparkFun:CAP0805
- removed PAD1, PAD10, PAD11, PAD12, PAD13, PAD14, PAD15, PAD16, PAD2, PAD3, PAD4, PAD5, PAD6, PAD7, PAD8, PAD9: (no value), wirepad:SMD2
- removed U2: STP16CP05SO-24, Synapseware:STP16CP05SO-24
- added LED1, LED2, LED3, LED4: (no value), wirepad:SMD2
- added R2, R4, R5: 68, SparkFun:RESISTOR0805-RES
- R1: value (none) -> 68
- Y1: value FA-128 -> (none); device crystal:FA-128 -> SparkFun-FreqCtrl:CRYSTAL5X3
Connections:
- net RXD renamed RX
- net TXD renamed TX
- removed net N$11: PAD7.P, U2./OUT6
- removed net N$13: PAD8.P, U2./OUT7
- removed net N$14: PAD9.P, U2./OUT8
- removed net N$15: PAD10.P, U2./OUT9
- removed net N$16: PAD11.P, U2./OUT10
- removed net N$17: PAD12.P, U2./OUT11
- removed net N$18: PAD13.P, U2./OUT12
- removed net N$19: PAD14.P, U2./OUT13
- removed net N$20: PAD15.P, U2./OUT14
- removed net N$21: PAD16.P, U2./OUT15
- removed net N$37: PAD5.P, U2./OUT4
- removed net N$5: PAD2.P, U2./OUT1
- removed net N$6: PAD3.P, U2./OUT2
- removed net N$7: PAD4.P, U2./OUT3
- removed net N$8: PAD6.P, U2./OUT5
- new net LED1: IC1.(AIN0)PB0, R1.2
- new net LED2: IC1.(AIN1)PB1, R2.2
- new net LED3: IC1.PB2, R4.2
- new net LED4: IC1.(OCI)PB3, R5.2
- new net N$2: LED3.P, R4.1
- new net N$3: LED2.P, R2.1
- net /OE: no longer U2./OE
- net 5V: no longer C3.1, U2.VDD
- net CLK: no longer U2.CLK
- net DATA: no longer U2.SDI
- net GND: no longer C3.2, R1.1, U2.GND
- net LE: no longer U2.LE
- net N$1: now also LED4.P, R5.1; no longer R1.2, U2.R-EXT
- net N$4: now also LED1.P, R1.1; no longer PAD1.P, U2./OUT0
Other:
- note removed: "/OE"
- note removed: "CLOCK"
- note removed: "DATA"
- note removed: "LE"
- note removed: "PWR_SENSE"
- note removed: "RX"
- note removed: "TX"
- moved on the sheet: R1
